File: Mouse/Mouse.kicad_pcb (KiCad board)
At the start: 2 copper layers, 21 parts

Commit message: updated footprints
Parts:
- added J1: Conn_01x05_Male, Mouse:JST_Conn, B.Cu at (130.5, 81.5)
- added U1: Left click, Mouse:SPDT_Switch, B.Cu at (167.3, 66.4)
- added U2: Middle click, Mouse:SPDT_Switch, B.Cu at (167.3, 80.3)
- added U3: Right Click, Mouse:SPDT_Switch, B.Cu at (174.2, 66.4)
- added U4: LQ1, Mouse:LQ1, B.Cu at (179.7, 78.7)
- added U5: Optical_Sensor, Mouse:Sensor, F.Cu at (133.6, 75.4)
- LD1, LD2: moved to B.Cu
- moved LD1 55.3 mm to (128.6, 51.6)
- moved LD2 50.1 mm to (135.6, 42.8)
Other:
- board outline added: 28 x 9.8 mm
