File: Mouse/Mouse.sch (KiCad schematic (older format))
At the start: 27 parts, among them J1 Conn_01x05_Male, U1 Left click, U2 Middle click, U3 Right Click

Commit message: added footprints
Parts:
- C11, C12, C8, C9: footprint (none) -> Capacitor_SMD:C_0402_1005Metric_Pad0.74x0.62mm_HandSolder
- C13: renamed from C?; value C13 -> C; footprint (none) -> Capacitor_SMD:C_0402_1005Metric_Pad0.74x0.62mm_HandSolder
- C14: footprint (none) -> Capacitor_SMD:C_0201_0603Metric_Pad0.64x0.40mm_HandSolder
- C15, C16: footprint (none) -> Capacitor_SMD:C_01005_0402Metric_Pad0.57x0.30mm_HandSolder
- LD1: footprint LED_THT:LED_D5.0mm_IRGrey -> LED_THT:LED_D2.0mm_W4.0mm_H2.8mm_FlatTop
- LD2: footprint LED_THT:LED_D5.0mm_IRGrey -> LED_THT:LED_D5.0mm_Horizontal_O6.35mm_Z15.0mm
- R10, R11, R12, R13, R15, R16, R17, R7, R8, R9: footprint (none) -> Resistor_SMD:R_01005_0402Metric_Pad0.57x0.30mm_HandSolder
- R14: footprint (none) -> Resistor_SMD:R_0402_1005Metric_Pad0.72x0.64mm_HandSolder
- gave numbers to parts that had none: 2
Connections:
- wire segments 44 -> 45

Commit message: updated footprints
Parts:
- J1: footprint (none) -> Mouse:JST_Conn
- U1, U2, U3: footprint (none) -> Mouse:SPDT_Switch; symbol optical~mouse:switch -> Optical_Mouse:switch
- U4: footprint (none) -> Mouse:LQ1; symbol optical~mouse:LQ -> Optical_Mouse:LQ
- U5: footprint (none) -> Mouse:Sensor; symbol optical~mouse:Optical_Sensor -> Optical_Mouse:Optical_Sensor
Changed lines of the file:
@@
 $EndDescr
 $Comp
-L optical~mouse:switch U1
+L Optical_Mouse:switch U1
 U 1 1 62F7695E
 P 2550 1550
 F 0 "U1" H 2678 1596 50  0000 L CNN
 F 1 "Left click" H 2678 1505 50  0000 L CNN
-F 2 "" H 2800 1650 50  0001 C CNN
+F 2 "Mouse:SPDT_Switch" H 2800 1650 50  0001 C CNN
 F 3 "" H 2800 1650 50  0001 C CNN
 	1    2550 1550
@@
 F 0 "J1" H 1008 5181 50  0000 C CNN
 F 1 "Conn_01x05_Male" H 1008 5090 50  0000 C CNN
-F 2 "" H 900 4800 50  0001 C CNN
+F 2 "Mouse:JST_Conn" H 900 4800 50  0001 C CNN
 F 3 "~" H 900 4800 50  0001 C CNN
 	1    900  4800
@@
 	550  7250 2850 7250
 $Comp
-L optical~mouse:switch U3
+L Optical_Mouse:switch U3
 U 1 1 62F77846
 P 1200 1550
 F 0 "U3" H 1328 1596 50  0000 L CNN
 F 1 "Right Click" H 1328 1505 50  0000 L CNN
-F 2 "" H 1450 1650 50  0001 C CNN
+F 2 "Mouse:SPDT_Switch" H 1450 1650 50  0001 C CNN
 F 3 "" H 1450 1650 50  0001 C CNN
 	1    1200 1550
@@
 $EndComp
 $Comp
-L optical~mouse:switch U2
+L Optical_Mouse:switch U2
 U 1 1 62F76FC9
 P 1150 2600
 F 0 "U2" V 1046 2878 50  0000 L CNN
 F 1 "Middle click" V 1137 2878 50  0000 L CNN
-F 2 "" H 1400 2700 50  0001 C CNN
+F 2 "Mouse:SPDT_Switch" H 1400 2700 50  0001 C CNN
 F 3 "" H 1400 2700 50  0001 C CNN
 	1    1150 2600
@@
 Pin_2
 $Comp
-L optical~mouse:LQ U4
+L Optical_Mouse:LQ U4
 U 1 1 62F9C524
 P 1150 6500
 F 0 "U4" H 1228 6461 50  0000 L CNN
 F 1 "LQ1" H 1228 6370 50  0000 L CNN
-F 2 "" H 1150 6600 50  0001 C CNN
+F 2 "Mouse:LQ1" H 1150 6600 50  0001 C CNN
 F 3 "" H 1150 6600 50  0001 C CNN
 	1    1150 6500
@@
 	2500 3650 2700 3650
 $Comp
-L optical~mouse:Optical_Sensor U5
+L Optical_Mouse:Optical_Sensor U5
 U 1 1 62F7519C
 P 1800 3450
 F 0 "U5" H 1750 3150 50  0000 L CNN
 F 1 "Optical_Sensor" H 1550 3950 50  0000 L CNN
-F 2 "" H 1800 3450 50  0001 C CNN
+F 2 "Mouse:Sensor" H 1800 3450 50  0001 C CNN
 F 3 "" H 1800 3450 50  0001 C CNN
 	1    1800 3450
