File: Mouse.kicad_pcb (KiCad board)
At the start: 2 copper layers, 39 x 78 mm, 31 parts, among them J1 Conn_01x05_Male, SW1 Left click, SW2 Right Click, SW3 Middle click, U1 Optical_Sensor

Commit message: Schematic Correction
Parts:
- C11, C13: value C -> C NC
- C12, C15: value C -> C 0.1uF
- C14: value C -> C 4.7uF
- C8, C9: value C -> C 0.01uF
- LQ1: value LQ1 -> EL
- R11: value 330_M_click -> R 303
- R12: value 330 LD2 resistor -> R 330
- R17: value R -> R NC
Connections:
- R7 pad 1: Pin_8 -> D-
